Commit message: is motor neuron breaking

File: body.urdf (robot description, URDF)
Before this commit: robot robot, 7 links, 6 joints
Links:
- removed link Link0
- removed link Link1
- removed link Link2
- removed link Link3
- removed link Link4
- removed link Link5
- removed link Link6
- added link BackLeg, mass 1; collision box size=1 1 1; visual box size=1 1 1
- added link FrontLeg, mass 1; collision box size=1 1 1; visual box size=1 1 1
- added link Torso, mass 1; collision box size=1 1 1; visual box size=1 1 1
Joints:
- removed joint Link0_Link1
- removed joint Link1_Link2
- removed joint Link2_Link3
- removed joint Link3_Link4
- removed joint Link4_Link5
- removed joint Link5_Link6
- added joint Torso_BackLeg: type revolute, parent Torso, child BackLeg, origin xyz=1 0 1 rpy=0 0 0, axis 0 1 0, limit lower=-3.14159 upper=3.14159 effort=0.0 velocity=0.0
- added joint Torso_FrontLeg: type revolute, parent Torso, child FrontLeg, origin xyz=2 0 1 rpy=0 0 0, axis 0 1 0, limit lower=-3.14159 upper=3.14159 effort=0.0 velocity=0.0

File: simple.urdf (robot description, URDF)
Before this commit: robot robot, 3 links, 2 joints
Links:
- removed link Backleg
- removed link Frontleg
- added link BackLeg, mass 1; collision box size=1 1 1; visual box size=1 1 1
- added link FrontLeg, mass 1; collision box size=1 1 1; visual box size=1 1 1
Joints:
- removed joint Torso_Backleg
- removed joint Torso_Frontleg
- added joint Torso_BackLeg: type revolute, parent Torso, child BackLeg, origin xyz=1 0 1 rpy=0 0 0, axis 0 1 0, limit lower=-3.14159 upper=3.14159 effort=0.0 velocity=0.0
- added joint Torso_FrontLeg: type revolute, parent Torso, child FrontLeg, origin xyz=2 0 1 rpy=0 0 0, axis 0 1 0, limit lower=-3.14159 upper=3.14159 effort=0.0 velocity=0.0

Commit message: a6

File: body.urdf (robot description, URDF)
Before this commit: robot robot, 3 links, 2 joints
Links:
- removed link BackLeg
- removed link FrontLeg
- removed link Torso
- added link Head, mass 1; collision box size=2 2 2; visual box size=2 2 2
- added link Link0, mass 1; collision box size=1 3 3; visual box size=1 3 3
- added link Link1, mass 1; collision box size=5 3 3; visual box size=5 3 3
- added link Link2, mass 1; collision box size=1 4 5; visual box size=1 4 5
- added link Link3, mass 1; collision box size=1 4 1; visual box size=1 4 1
- added link Link4, mass 1; collision box size=3 1 2; visual box size=3 1 2
- added link Link5, mass 1; collision box size=2 3 4; visual box size=2 3 4
- added link Link6, mass 1; collision box size=4 5 1; visual box size=4 5 1
Joints:
- removed joint Torso_BackLeg
- removed joint Torso_FrontLeg
- added joint Head_Link0: type revolute, parent Head, child Link0, origin xyz=-10 19.0 2.5 rpy=0 0 0, axis 0 0 1, limit lower=-3.14159 upper=3.14159 effort=0.0 velocity=0.0
- added joint Link0_Link1: type revolute, parent Link0, child Link1, origin xyz=0 -3 0 rpy=0 0 0, axis 0 0 1, limit lower=-3.14159 upper=3.14159 effort=0.0 velocity=0.0
- added joint Link1_Link2: type revolute, parent Link1, child Link2, origin xyz=0 -3 0 rpy=0 0 0, axis 0 0 1, limit lower=-3.14159 upper=3.14159 effort=0.0 velocity=0.0
- added joint Link2_Link3: type revolute, parent Link2, child Link3, origin xyz=0 -4 0 rpy=0 0 0, axis 0 0 1, limit lower=-3.14159 upper=3.14159 effort=0.0 velocity=0.0
- added joint Link3_Link4: type revolute, parent Link3, child Link4, origin xyz=0 -4 0 rpy=0 0 0, axis 0 0 1, limit lower=-3.14159 upper=3.14159 effort=0.0 velocity=0.0
- added joint Link4_Link5: type revolute, parent Link4, child Link5, origin xyz=0 -1 0 rpy=0 0 0, axis 0 0 1, limit lower=-3.14159 upper=3.14159 effort=0.0 velocity=0.0
- added joint Link5_Link6: type revolute, parent Link5, child Link6, origin xyz=0 -3 0 rpy=0 0 0, axis 0 0 1, limit lower=-3.14159 upper=3.14159 effort=0.0 velocity=0.0

File: simple.urdf (robot description, URDF)
Before this commit: robot robot, 13 links, 12 joints
Links:
- removed link LeftLeg
- removed link LeftLeg2
- removed link LeftLeg3
- removed link LeftLowerLeg
- removed link LeftLowerLeg2
- removed link LeftLowerLeg3
- removed link RightLeg
- removed link RightLeg2
- removed link RightLeg3
- removed link RightLowerLeg
- removed link RightLowerLeg2
- removed link RightLowerLeg3
- added link Torso1, mass 1; collision box size=1.224100101726435 1.6766727190284265 2.924671156546345; visual box size=1.224100101726435 1.6766727190284265 2.924671156546345
- added link Torso2, mass 1; collision box size=1.2008910080800483 2.941341282151426 2.8838277426088164; visual box size=1.2008910080800483 2.941341282151426 2.8838277426088164
- added link Torso3, mass 1; collision box size=2.5699573463099457 1.9437967924915651 1.4054651904760056; visual box size=2.5699573463099457 1.9437967924915651 1.4054651904760056
- added link Torso4, mass 1; collision box size=1.9999749052512372 1.7841285079858 1.865389721329019; visual box size=1.9999749052512372 1.7841285079858 1.865389721329019
- added link Torso5, mass 1; collision box size=1.1808011175007722 2.6368671917244946 1.179597812528219; visual box size=1.1808011175007722 2.6368671917244946 1.179597812528219
- added link Torso6, mass 1; collision box size=2.1414305715627657 2.1752186676442213 1.1290098381433749; visual box size=2.1414305715627657 2.1752186676442213 1.1290098381433749
- link Torso: geometry collision box size=2.6952214071644818 2.8030933373978035 1.2259411540964076; visual box size=2.6952214071644818 2.8030933373978035 1.2259411540964076
Joints:
- removed joint LeftLeg2_LeftLowerLeg2
- removed joint LeftLeg3_LeftLowerLeg3
- removed joint LeftLeg_LeftLowerLeg
- removed joint RightLeg2_RightLowerLeg2
- removed joint RightLeg3_RightLowerLeg3
- removed joint RightLeg_RightLowerLeg
- removed joint Torso_LeftLeg
- removed joint Torso_LeftLeg2
- removed joint Torso_LeftLeg3
- removed joint Torso_RightLeg
- removed joint Torso_RightLeg2
- removed joint Torso_RightLeg3
- added joint Torso10_Torso11: type revolute, parent Torso10, child Torso11, origin xyz=0 0.8383363595142133 0 rpy=0 0 0, axis 1 0 0, limit lower=-3.14159 upper=3.14159 effort=0.0 velocity=0.0
- added joint Torso11_Torso12: type revolute, parent Torso11, child Torso12, origin xyz=0 0.8383363595142133 0 rpy=0 0 0, axis 1 0 0, limit lower=-3.14159 upper=3.14159 effort=0.0 velocity=0.0
- added joint Torso1_Torso2: type revolute, parent Torso1, child Torso2, origin xyz=0 0.8383363595142133 0 rpy=0 0 0, axis 1 0 0, limit lower=-3.14159 upper=3.14159 effort=0.0 velocity=0.0
- added joint Torso2_Torso3: type revolute, parent Torso2, child Torso3, origin xyz=0 0.8383363595142133 0 rpy=0 0 0, axis 1 0 0, limit lower=-3.14159 upper=3.14159 effort=0.0 velocity=0.0
- added joint Torso3_Torso4: type revolute, parent Torso3, child Torso4, origin xyz=0 0.8383363595142133 0 rpy=0 0 0, axis 1 0 0, limit lower=-3.14159 upper=3.14159 effort=0.0 velocity=0.0
- added joint Torso4_Torso5: type revolute, parent Torso4, child Torso5, origin xyz=0 0.8383363595142133 0 rpy=0 0 0, axis 1 0 0, limit lower=-3.14159 upper=3.14159 effort=0.0 velocity=0.0
- added joint Torso5_Torso6: type revolute, parent Torso5, child Torso6, origin xyz=0 0.8383363595142133 0 rpy=0 0 0, axis 1 0 0, limit lower=-3.14159 upper=3.14159 effort=0.0 velocity=0.0
- added joint Torso6_Torso7: type revolute, parent Torso6, child Torso7, origin xyz=0 0.8383363595142133 0 rpy=0 0 0, axis 1 0 0, limit lower=-3.14159 upper=3.14159 effort=0.0 velocity=0.0
- added joint Torso7_Torso8: type revolute, parent Torso7, child Torso8, origin xyz=0 0.8383363595142133 0 rpy=0 0 0, axis 1 0 0, limit lower=-3.14159 upper=3.14159 effort=0.0 velocity=0.0
- added joint Torso8_Torso9: type revolute, parent Torso8, child Torso9, origin xyz=0 0.8383363595142133 0 rpy=0 0 0, axis 1 0 0, limit lower=-3.14159 upper=3.14159 effort=0.0 velocity=0.0
- added joint Torso9_Torso10: type revolute, parent Torso9, child Torso10, origin xyz=0 0.8383363595142133 0 rpy=0 0 0, axis 1 0 0, limit lower=-3.14159 upper=3.14159 effort=0.0 velocity=0.0
- added joint Torso_Torso1: type revolute, parent Torso, child Torso1, origin xyz=0 1.4015466686989018 0.6129705770482038 rpy=0 0 0, axis 1 0 0, limit lower=-3.14159 upper=3.14159 effort=0.0 velocity=0.0

Commit message: some cleaning in solution

File: body.urdf (robot description, URDF)
Before this commit: robot robot, 8 links, 7 joints
Links:
- link Head: geometry collision box size=2 3 1; visual box size=2 3 1
- link Link0: geometry collision box size=4 4 4; visual box size=4 4 4
- link Link1: geometry collision box size=4 2 3; visual box size=4 2 3
- link Link2: geometry collision box size=2 5 4; visual box size=2 5 4
- link Link3: geometry collision box size=2 5 4; visual box size=2 5 4
- link Link4: geometry collision box size=4 4 3; visual box size=4 4 3
- link Link5: geometry collision box size=5 4 5; visual box size=5 4 5
- link Link6: geometry collision box size=2 2 5; visual box size=2 2 5
Joints:
- joint Head_Link0: origin xyz=-10 19.0 2.5 rpy=0 0 0 -> xyz=-10 18.5 2.5 rpy=0 0 0
- joint Link0_Link1: origin xyz=0 -3 0 rpy=0 0 0 -> xyz=0 -4 0 rpy=0 0 0
- joint Link1_Link2: origin xyz=0 -3 0 rpy=0 0 0 -> xyz=0 -2 0 rpy=0 0 0
- joint Link2_Link3: origin xyz=0 -4 0 rpy=0 0 0 -> xyz=0 -5 0 rpy=0 0 0
- joint Link3_Link4: origin xyz=0 -4 0 rpy=0 0 0 -> xyz=0 -5 0 rpy=0 0 0
- joint Link4_Link5: origin xyz=0 -1 0 rpy=0 0 0 -> xyz=0 -4 0 rpy=0 0 0
- joint Link5_Link6: origin xyz=0 -3 0 rpy=0 0 0 -> xyz=0 -4 0 rpy=0 0 0

Commit message: stuff

File: body.urdf (robot description, URDF)
Before this commit: robot robot, 8 links, 7 joints
Links:
- removed link Head
- removed link Link0
- removed link Link1
- removed link Link2
- removed link Link3
- removed link Link4
- removed link Link5
- removed link Link6
- added link base, mass 1; collision box size=1 1 1; visual box size=1 1 1
Joints:
- removed joint Head_Link0
- removed joint Link0_Link1
- removed joint Link1_Link2
- removed joint Link2_Link3
- removed joint Link3_Link4
- removed joint Link4_Link5
- removed joint Link5_Link6

Commit message: a7

File: body.urdf (robot description, URDF)
Before this commit: robot robot, 9 links, 8 joints
Links:
- link limb0: geometry collision box size=0.6666666666666666 1 0.5; visual box size=0.6666666666666666 1 0.5
- link limb1: geometry collision box size=0.2 0.5 0.2; visual box size=0.2 0.5 0.2
- link limb2: geometry collision box size=0.2 0.2 0.4; visual box size=0.2 0.2 0.4
- link limb3: geometry collision box size=0.2 0.5 0.2; visual box size=0.2 0.5 0.2
- link limb4: geometry collision box size=0.2 0.2 0.4; visual box size=0.2 0.2 0.4
- link limb5: geometry collision box size=0.2 0.5 0.2; visual box size=0.2 0.5 0.2
- link limb6: geometry collision box size=0.2 0.2 0.4; visual box size=0.2 0.2 0.4
- link limb7: geometry collision box size=0.2 0.5 0.2; visual box size=0.2 0.5 0.2
- link limb8: geometry collision box size=0.2 0.2 0.4; visual box size=0.2 0.2 0.4
Joints:
- joint limb0_limb1: origin xyz=0.0 -0.0 0.8862819657069074 rpy=0 0 0 -> xyz=-1.5 -0.5 0.45 rpy=0 0 0
- joint limb0_limb3: origin xyz=0.3 -0.3 0.8862819657069074 rpy=0 0 0 -> xyz=-0.5 -0.5 0.45 rpy=0 0 0
- joint limb0_limb5: origin xyz=0.0 0.0 0.8862819657069074 rpy=0 0 0 -> xyz=-1.5 0.5 0.45 rpy=0 0 0
- joint limb0_limb7: origin xyz=0.15 0.15 0.8862819657069074 rpy=0 0 0 -> xyz=-0.5 0.5 0.45 rpy=0 0 0
- joint limb1_limb2: axis 1 1 0 -> 0 0 1; origin xyz=0.0 -0.0 0.8862819657069074 rpy=0 0 0 -> xyz=0 -0.5 0 rpy=0 0 0
- joint limb3_limb4: axis 1 1 0 -> 0 0 1; origin xyz=0.3 -0.3 0.8862819657069074 rpy=0 0 0 -> xyz=0 -0.5 0 rpy=0 0 0
- joint limb5_limb6: axis 1 1 0 -> 0 0 1; origin xyz=0.0 0.0 0.8862819657069074 rpy=0 0 0 -> xyz=0 0.5 0 rpy=0 0 0
- joint limb7_limb8: axis 1 1 0 -> 0 0 1; origin xyz=0.3 0.3 0.8862819657069074 rpy=0 0 0 -> xyz=0 0.5 0 rpy=0 0 0

Commit message: misc

File: body.urdf (robot description, URDF)
Before this commit: robot robot, 9 links, 8 joints
Links:
- link limb0: geometry collision box size=0.4300253909340138 0.4754118197311067 0.4369068227782664; visual box size=0.4300253909340138 0.4754118197311067 0.4369068227782664
- link limb1: geometry collision box size=0.4300253909340138 0.4754118197311067 0.4369068227782664; visual box size=0.4300253909340138 0.4754118197311067 0.4369068227782664
- link limb2: geometry collision box size=0.4300253909340138 0.4754118197311067 0.4369068227782664; visual box size=0.4300253909340138 0.4754118197311067 0.4369068227782664
- link limb3: geometry collision box size=0.4300253909340138 0.4754118197311067 0.4369068227782664; visual box size=0.4300253909340138 0.4754118197311067 0.4369068227782664
- link limb4: geometry collision box size=0.4300253909340138 0.4754118197311067 0.4369068227782664; visual box size=0.4300253909340138 0.4754118197311067 0.4369068227782664
- link limb5: geometry collision box size=0.4300253909340138 0.4754118197311067 0.4369068227782664; visual box size=0.4300253909340138 0.4754118197311067 0.4369068227782664
- link limb6: geometry collision box size=0.4300253909340138 0.4754118197311067 0.4369068227782664; visual box size=0.4300253909340138 0.4754118197311067 0.4369068227782664
- link limb7: geometry collision box size=0.4300253909340138 0.4754118197311067 0.4369068227782664; visual box size=0.4300253909340138 0.4754118197311067 0.4369068227782664
- link limb8: geometry collision box size=0.4300253909340138 0.4754118197311067 0.4369068227782664; visual box size=0.4300253909340138 0.4754118197311067 0.4369068227782664
Joints:
- joint limb0_limb1: origin xyz=-1.5 -0.5 0.45 rpy=0 0 0 -> xyz=0.0 -0.0 0.4369068227782664 rpy=0 0 0
- joint limb0_limb3: origin xyz=-0.5 -0.5 0.45 rpy=0 0 0 -> xyz=0.3 -0.3 0.4369068227782664 rpy=0 0 0
- joint limb0_limb5: origin xyz=-1.5 0.5 0.45 rpy=0 0 0 -> xyz=0.0 0.0 0.4369068227782664 rpy=0 0 0
- joint limb0_limb7: origin xyz=-0.5 0.5 0.45 rpy=0 0 0 -> xyz=0.15 0.15 0.4369068227782664 rpy=0 0 0
- joint limb1_limb2: axis 0 0 1 -> 1 1 0; origin xyz=0 -0.5 0 rpy=0 0 0 -> xyz=0.0 -0.0 0.4369068227782664 rpy=0 0 0
- joint limb3_limb4: axis 0 0 1 -> 1 1 0; origin xyz=0 -0.5 0 rpy=0 0 0 -> xyz=0.3 -0.3 0.4369068227782664 rpy=0 0 0
- joint limb5_limb6: axis 0 0 1 -> 1 1 0; origin xyz=0 0.5 0 rpy=0 0 0 -> xyz=0.0 0.0 0.4369068227782664 rpy=0 0 0
- joint limb7_limb8: axis 0 0 1 -> 1 1 0; origin xyz=0 0.5 0 rpy=0 0 0 -> xyz=0.3 0.3 0.4369068227782664 rpy=0 0 0

Commit message: working 3D body generator

File: body.urdf (robot description, URDF)
Before this commit: robot robot, 9 links, 8 joints
Links:
- added link limb10, mass 1; collision box size=0.11398672301070159 0.4318573652522619 0.58920650858361; visual box size=0.11398672301070159 0.4318573652522619 0.58920650858361
- added link limb11, mass 1; collision box size=0.2 0.5 0.2; visual box size=0.2 0.5 0.2
- added link limb12, mass 1; collision box size=0.15281873226544979 0.4978920951212295 0.4433438627287204; visual box size=0.15281873226544979 0.4978920951212295 0.4433438627287204
- added link limb13, mass 1; collision box size=0.2 0.5 0.2; visual box size=0.2 0.5 0.2
- added link limb14, mass 1; collision box size=0.1702200221621705 0.43671559061120224 0.347847773172721; visual box size=0.1702200221621705 0.43671559061120224 0.347847773172721
- added link limb15, mass 1; collision box size=0.2 0.5 0.2; visual box size=0.2 0.5 0.2
- added link limb16, mass 1; collision box size=0.23232385749626303 0.4744083430838929 0.1625755470612773; visual box size=0.23232385749626303 0.4744083430838929 0.1625755470612773
- added link limb17, mass 1; collision box size=0.2 0.5 0.2; visual box size=0.2 0.5 0.2
- added link limb18, mass 1; collision box size=0.16330578027834877 0.34908190441727044 0.19777351932726392; visual box size=0.16330578027834877 0.34908190441727044 0.19777351932726392
- added link limb19, mass 1; collision box size=0.2 0.5 0.2; visual box size=0.2 0.5 0.2
- added link limb20, mass 1; collision box size=0.13998439769590354 0.32872669001325494 0.7189710482094831; visual box size=0.13998439769590354 0.32872669001325494 0.7189710482094831
- added link limb21, mass 1; collision box size=0.2 0.5 0.2; visual box size=0.2 0.5 0.2
- added link limb22, mass 1; collision box size=0.24496856575433784 0.43949862739077444 0.37306862438049104; visual box size=0.24496856575433784 0.43949862739077444 0.37306862438049104
- added link limb23, mass 1; collision box size=0.2 0.5 0.2; visual box size=0.2 0.5 0.2
- added link limb24, mass 1; collision box size=0.2145098166777923 0.4634492364504299 0.4727860809713559; visual box size=0.2145098166777923 0.4634492364504299 0.4727860809713559
- added link limb25, mass 1; collision box size=0.26216037943528536 0.4228870777327535 0.5851006032251239; visual box size=0.26216037943528536 0.4228870777327535 0.5851006032251239
- added link limb9, mass 1; collision box size=0.2 0.5 0.2; visual box size=0.2 0.5 0.2
- link limb0: geometry collision box size=6 1 0.5; visual box size=6 1 0.5
- link limb1: geometry collision box size=0.2 0.5 0.2; visual box size=0.2 0.5 0.2
- link limb2: geometry collision box size=0.13323885736747101 0.483466825708936 0.6486339551805521; visual box size=0.13323885736747101 0.483466825708936 0.6486339551805521
- link limb3: geometry collision box size=0.2 0.5 0.2; visual box size=0.2 0.5 0.2
- link limb4: geometry collision box size=0.23540828463586774 0.37711922606718223 0.5527653916435739; visual box size=0.23540828463586774 0.37711922606718223 0.5527653916435739
- link limb5: geometry collision box size=0.2 0.5 0.2; visual box size=0.2 0.5 0.2
- link limb6: geometry collision box size=0.1736985145751206 0.3317656270496058 0.23801987773730146; visual box size=0.1736985145751206 0.3317656270496058 0.23801987773730146
- link limb7: geometry collision box size=0.2 0.5 0.2; visual box size=0.2 0.5 0.2
- link limb8: geometry collision box size=0.211911771017272 0.39631404509585455 0.4196470906662977; visual box size=0.211911771017272 0.39631404509585455 0.4196470906662977
Joints:
- added joint limb0_limb11: type revolute, parent limb0, child limb11, origin xyz=-0.5 -0.5 0.45 rpy=0 0 0, axis 0 1 0, limit lower=-3.14159 upper=3.14159 effort=0.0 velocity=0.0
- added joint limb0_limb13: type revolute, parent limb0, child limb13, origin xyz=-5.5 0.5 0.45 rpy=0 0 0, axis 0 1 0, limit lower=-3.14159 upper=3.14159 effort=0.0 velocity=0.0
- added joint limb0_limb15: type revolute, parent limb0, child limb15, origin xyz=-4.5 0.5 0.45 rpy=0 0 0, axis 0 1 0, limit lower=-3.14159 upper=3.14159 effort=0.0 velocity=0.0
- added joint limb0_limb17: type revolute, parent limb0, child limb17, origin xyz=-3.5 0.5 0.45 rpy=0 0 0, axis 0 1 0, limit lower=-3.14159 upper=3.14159 effort=0.0 velocity=0.0
- added joint limb0_limb19: type revolute, parent limb0, child limb19, origin xyz=-2.5 0.5 0.45 rpy=0 0 0, axis 0 1 0, limit lower=-3.14159 upper=3.14159 effort=0.0 velocity=0.0
- added joint limb0_limb21: type revolute, parent limb0, child limb21, origin xyz=-1.5 0.5 0.45 rpy=0 0 0, axis 0 1 0, limit lower=-3.14159 upper=3.14159 effort=0.0 velocity=0.0
- added joint limb0_limb23: type revolute, parent limb0, child limb23, origin xyz=-0.5 0.5 0.45 rpy=0 0 0, axis 0 1 0, limit lower=-3.14159 upper=3.14159 effort=0.0 velocity=0.0
- added joint limb0_limb25: type revolute, parent limb0, child limb25, origin xyz=-5.5 0 0.35 rpy=0 0 0, axis 0 0 1, limit lower=-3.14159 upper=3.14159 effort=0.0 velocity=0.0
- added joint limb0_limb9: type revolute, parent limb0, child limb9, origin xyz=-1.5 -0.5 0.45 rpy=0 0 0, axis 0 1 0, limit lower=-3.14159 upper=3.14159 effort=0.0 velocity=0.0
- added joint limb11_limb12: type revolute, parent limb11, child limb12, origin xyz=0 -0.5 0 rpy=0 0 0, axis 1 0 0, limit lower=-3.14159 upper=3.14159 effort=0.0 velocity=0.0
- added joint limb13_limb14: type revolute, parent limb13, child limb14, origin xyz=0 0.5 0 rpy=0 0 0, axis 1 0 0, limit lower=-3.14159 upper=3.14159 effort=0.0 velocity=0.0
- added joint limb15_limb16: type revolute, parent limb15, child limb16, origin xyz=0 0.5 0 rpy=0 0 0, axis 1 0 0, limit lower=-3.14159 upper=3.14159 effort=0.0 velocity=0.0
- added joint limb17_limb18: type revolute, parent limb17, child limb18, origin xyz=0 0.5 0 rpy=0 0 0, axis 1 0 0, limit lower=-3.14159 upper=3.14159 effort=0.0 velocity=0.0
- added joint limb19_limb20: type revolute, parent limb19, child limb20, origin xyz=0 0.5 0 rpy=0 0 0, axis 1 0 0, limit lower=-3.14159 upper=3.14159 effort=0.0 velocity=0.0
- added joint limb21_limb22: type revolute, parent limb21, child limb22, origin xyz=0 0.5 0 rpy=0 0 0, axis 1 0 0, limit lower=-3.14159 upper=3.14159 effort=0.0 velocity=0.0
- added joint limb23_limb24: type revolute, parent limb23, child limb24, origin xyz=0 0.5 0 rpy=0 0 0, axis 1 0 0, limit lower=-3.14159 upper=3.14159 effort=0.0 velocity=0.0
- added joint limb9_limb10: type revolute, parent limb9, child limb10, origin xyz=0 -0.5 0 rpy=0 0 0, axis 1 0 0, limit lower=-3.14159 upper=3.14159 effort=0.0 velocity=0.0
- joint limb0_limb1: axis 1 1 0 -> 0 1 0; origin xyz=0.0 -0.0 0.4369068227782664 rpy=0 0 0 -> xyz=-5.5 -0.5 0.45 rpy=0 0 0
- joint limb0_limb3: axis 1 1 0 -> 0 1 0; origin xyz=0.3 -0.3 0.4369068227782664 rpy=0 0 0 -> xyz=-4.5 -0.5 0.45 rpy=0 0 0
- joint limb0_limb5: axis 1 1 0 -> 0 1 0; origin xyz=0.0 0.0 0.4369068227782664 rpy=0 0 0 -> xyz=-3.5 -0.5 0.45 rpy=0 0 0
- joint limb0_limb7: axis 1 1 0 -> 0 1 0; origin xyz=0.15 0.15 0.4369068227782664 rpy=0 0 0 -> xyz=-2.5 -0.5 0.45 rpy=0 0 0
- joint limb1_limb2: axis 1 1 0 -> 1 0 0; origin xyz=0.0 -0.0 0.4369068227782664 rpy=0 0 0 -> xyz=0 -0.5 0 rpy=0 0 0
- joint limb3_limb4: axis 1 1 0 -> 1 0 0; origin xyz=0.3 -0.3 0.4369068227782664 rpy=0 0 0 -> xyz=0 -0.5 0 rpy=0 0 0
- joint limb5_limb6: axis 1 1 0 -> 1 0 0; origin xyz=0.0 0.0 0.4369068227782664 rpy=0 0 0 -> xyz=0 -0.5 0 rpy=0 0 0
- joint limb7_limb8: axis 1 1 0 -> 1 0 0; origin xyz=0.3 0.3 0.4369068227782664 rpy=0 0 0 -> xyz=0 -0.5 0 rpy=0 0 0
