Commit message: a8 completed

File: body.urdf (robot description, URDF)
Before this commit: robot robot, 26 links, 25 joints
Links:
- removed link limb18
- removed link limb19
- removed link limb20
- removed link limb21
- removed link limb22
- removed link limb23
- removed link limb24
- removed link limb25
- link limb0: geometry collision box size=4 1 0.5; visual box size=4 1 0.5
- link limb10: geometry collision box size=0.2 0.3 0.2; visual box size=0.2 0.3 0.2
- link limb12: geometry collision box size=0.2 0.3 0.2; visual box size=0.2 0.3 0.2
- link limb14: geometry collision box size=0.2 0.3 0.2; visual box size=0.2 0.3 0.2
- link limb16: geometry collision box size=0.2 0.3 0.2; visual box size=0.2 0.3 0.2
- link limb17: geometry collision box size=0.13828543083076847 0.316093596916544 0.7307656740103828; visual box size=0.13828543083076847 0.316093596916544 0.7307656740103828
- link limb2: geometry collision box size=0.2 0.3 0.2; visual box size=0.2 0.3 0.2
- link limb4: geometry collision box size=0.2 0.3 0.2; visual box size=0.2 0.3 0.2
- link limb6: geometry collision box size=0.2 0.3 0.2; visual box size=0.2 0.3 0.2
- link limb8: geometry collision box size=0.2 0.3 0.2; visual box size=0.2 0.3 0.2
Joints:
- removed joint limb0_limb19
- removed joint limb0_limb21
- removed joint limb0_limb23
- removed joint limb0_limb25
- removed joint limb17_limb18
- removed joint limb19_limb20
- removed joint limb21_limb22
- removed joint limb23_limb24
- joint limb0_limb1: origin xyz=-5.5 -0.5 0.45 rpy=0 0 0 -> xyz=-3.5 -0.5 0.45 rpy=0 0 0
- joint limb0_limb11: origin xyz=-0.5 -0.5 0.45 rpy=0 0 0 -> xyz=-2.5 0.5 0.45 rpy=0 0 0
- joint limb0_limb13: origin xyz=-5.5 0.5 0.45 rpy=0 0 0 -> xyz=-1.5 0.5 0.45 rpy=0 0 0
- joint limb0_limb15: origin xyz=-4.5 0.5 0.45 rpy=0 0 0 -> xyz=-0.5 0.5 0.45 rpy=0 0 0
- joint limb0_limb17: axis 0 1 0 -> 0 0 1; origin xyz=-3.5 0.5 0.45 rpy=0 0 0 -> xyz=-3.5 0 0.35 rpy=0 0 0
- joint limb0_limb3: origin xyz=-4.5 -0.5 0.45 rpy=0 0 0 -> xyz=-2.5 -0.5 0.45 rpy=0 0 0
- joint limb0_limb5: origin xyz=-3.5 -0.5 0.45 rpy=0 0 0 -> xyz=-1.5 -0.5 0.45 rpy=0 0 0
- joint limb0_limb7: origin xyz=-2.5 -0.5 0.45 rpy=0 0 0 -> xyz=-0.5 -0.5 0.45 rpy=0 0 0
- joint limb0_limb9: origin xyz=-1.5 -0.5 0.45 rpy=0 0 0 -> xyz=-3.5 0.5 0.45 rpy=0 0 0
- joint limb11_limb12: origin xyz=0 -0.5 0 rpy=0 0 0 -> xyz=0 0.5 0 rpy=0 0 0
- joint limb9_limb10: origin xyz=0 -0.5 0 rpy=0 0 0 -> xyz=0 0.5 0 rpy=0 0 0
